Commit message: robot_localization

File: limo_description/urdf/limo_ackerman.xacro (robot description, xacro)
@@ -12,4 +12,5 @@
     <xacro:property name="base_z_size" value="0.10" />
     <xacro:property name="wheelbase" value="0.2"/>
+    <!-- <xacro:property name="track" value="0.14"/> -->
     <xacro:property name="track" value="0.14"/>
     <xacro:property name="wheel_vertical_offset" value="-0.100998" />
